File: HW/esp12Board/esp12Board.kicad_pcb (KiCad board)
At the start: 2 copper layers, 50 x 50 mm, 49 parts, among them IC1 TPS54331DR, J1 Conn_01x07, J2 Conn_01x03, J3 Conn_02x05_Odd_Even, J4 Conn_01x02, J5 Conn_01x03, J6 Conn_01x03, J7 Conn_01x03, J8 Conn_01x03, Q1 S8050_SMD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

Commit message: update platta HW
Parts:
- C10: footprint Capacitor_SMD:C_0805_2012Metric_Pad1.15x1.40mm_HandSolder -> Capacitor_SMD:C_0603_1608Metric_Pad1.08x0.95mm_HandSolder
- C2, C4: value CP_Small -> 47uF; footprint Capacitor_THT:CP_Radial_D5.0mm_P2.50mm -> Capacitor_SMD:CP_Elec_5x5.7
- moved C2 2.50 mm to (38.0, 75.9)
- moved D1 1.00 mm to (44.5, 74.5)
- moved C4 0.75 mm to (39.8, 53.0)
- moved C5 0.75 mm to (31.8, 75.2)
- moved J6 0.34 mm to (78.0, 76.0)
- moved J2 0.22 mm to (78.0, 67.8)
- moved J5 0.22 mm to (78.0, 72.0)
Connections:
- IC1 pad 3: (no net) -> unconnected-(IC1-EN-Pad3)
- J1 pad 6: (no net) -> unconnected-(J1-Pin_6-Pad6)
- U1 pad 10: (no net) -> unconnected-(U1-MISO-Pad10)
- U1 pad 11: (no net) -> unconnected-(U1-IO9-Pad11)
- U1 pad 12: (no net) -> unconnected-(U1-IO10-Pad12)
- U1 pad 13: (no net) -> unconnected-(U1-MOSI-Pad13)
- U1 pad 14: (no net) -> unconnected-(U1-SCLK-Pad14)
- U1 pad 9: (no net) -> unconnected-(U1-CS0-Pad9)
Routing:
- net GND: track 36.7 -> 45.6 mm, vias 12 -> 13
- net +5V: track 66.4 -> 70.4 mm
- net VIN: track 17.1 -> 17.8 mm
Other:
- net class Default removed
- net class bigger removed
